File: RepRapLtd/Electronics/arduino-shield/arduino-shield.kicad_pcb (KiCad board)
At the start: 2 copper layers, 68.8 x 53.5 mm, 7 parts, among them J1 Conn_01x03, J2 Conn_01x03, J3 Conn_01x03, J4 Conn_01x03, J5 Conn_01x03, J6 Conn_01x03

Commit message: Added button connectors and LED connector to the Arduino shield.
Parts:
- removed A1: Arduino_UNO_R3_Shield, reprapltd-kicad:Arduino_UNO_R3_Shield
- removed J1, J2, J3, J4, J5, J6: Conn_01x03, Connector_PinHeader_2.54mm:PinHeader_1x03_P2.54mm_Vertical
Routing:
- net +5V: track 34.7 -> 0.00 mm
- net GND: track 31.9 -> 0.00 mm
- net Net-(A1-Pad9): track 8.54 -> 0.00 mm
- net Net-(A1-Pad13): track 8.54 -> 0.00 mm
- net Net-(A1-Pad12): track 8.54 -> 0.00 mm
- net Net-(A1-Pad10): track 8.54 -> 0.00 mm
- net Net-(A1-Pad14): track 8.54 -> 0.00 mm
- net Net-(A1-Pad11): track 8.54 -> 0.00 mm
- removed copper zone on F.Cu, net GND
Other:
- board outline removed

Commit message: 3-axis integrated design for all torques added.
Parts:
- added A1: Arduino_UNO_R3_Shield, reprapltd-kicad:Arduino_UNO_R3_Shield, F.Cu at (127.3, 119.7)
- added J1: Conn_01x03, Connector_PinHeader_2.54mm:PinHeader_1x03_P2.54mm_Vertical, F.Cu at (146.1, 110.5)
- added J10: Conn_01x02, Connector_PinHeader_2.54mm:PinHeader_1x02_P2.54mm_Vertical, F.Cu at (124.5, 76.2)
- added J2: Conn_01x03, Connector_PinHeader_2.54mm:PinHeader_1x03_P2.54mm_Vertical, F.Cu at (149.9, 110.5)
- added J3: Conn_01x03, Connector_PinHeader_2.54mm:PinHeader_1x03_P2.54mm_Vertical, F.Cu at (153.7, 110.5)
- added J4: Conn_01x03, Connector_PinHeader_2.54mm:PinHeader_1x03_P2.54mm_Vertical, F.Cu at (157.5, 110.5)
- added J5: Conn_01x03, Connector_PinHeader_2.54mm:PinHeader_1x03_P2.54mm_Vertical, F.Cu at (161.3, 110.5)
- added J6: Conn_01x03, Connector_PinHeader_2.54mm:PinHeader_1x03_P2.54mm_Vertical, F.Cu at (165.1, 110.5)
- added J7: Conn_01x02, Connector_PinHeader_2.54mm:PinHeader_1x02_P2.54mm_Vertical, F.Cu at (151.1, 78.7)
- added J8: Conn_01x02, Connector_PinHeader_2.54mm:PinHeader_1x02_P2.54mm_Vertical, F.Cu at (154.9, 78.7)
- added J9: Conn_01x02, Connector_PinHeader_2.54mm:PinHeader_1x02_P2.54mm_Vertical, F.Cu at (158.8, 78.7)
- added R1: 180R, Resistor_SMD:R_0805_2012Metric, F.Cu at (128.3, 77.8)
Routing:
- net +5V: track 0.00 -> 36.2 mm
- net Net-(A1-Pad9): track 0.00 -> 5.78 mm
- net Net-(A1-Pad28): track 0.00 -> 5.53 mm
- net Net-(A1-Pad19): track 0.00 -> 5.44 mm
- net Net-(A1-Pad10): track 0.00 -> 5.25 mm
- net Net-(A1-Pad17): track 0.00 -> 5.22 mm
- net Net-(A1-Pad14): track 0.00 -> 5.02 mm
- net Net-(A1-Pad18): track 0.00 -> 4.92 mm
- net Net-(A1-Pad11): track 0.00 -> 4.72 mm
- net Net-(A1-Pad13): track 0.00 -> 4.50 mm
- net Net-(A1-Pad12): track 0.00 -> 4.20 mm
- net Net-(J10-Pad2): track 0.00 -> 3.81 mm
- added copper zone on F.Cu, net GND
